File: GP2040-CE-DevBoard/outputs.kicad_sch (KiCad schematic)
At the start: 10 parts, among them J3 Debug, J4 RGB LED

Commit message: Updating schema and PCB design
Parts:
- added J5: qwiic, Connector_JST:JST_SH_BM04B-SRSS-TB_1x04-1MP_P1.00mm_Vertical, symbol Connector_Generic:Conn_01x04
Connections:
- net GND: now also J5.4 (Pin_4)
- new net +3V3: J5.3 (Pin_3)
- new net SCL: J5.1 (Pin_1)
- new net SDA: J5.2 (Pin_2)
Changed lines of the file:
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@@
+    (stroke (width 0) (type default) (color 0 0 0 0))
+  )
+  (wire (pts (xy 97.79 60.96) (xy 107.95 60.96))
     (stroke (width 0) (type default) (color 0 0 0 0))
   )
@@
     )
   )
+  (global_label "SDA" (shape input) (at 107.95 58.42 180) (fields_autoplaced)
+    (effects (font (size 1.27 1.27)) (justify right))
+    (property "Intersheet References" "${INTERSHEET_REFS}" (id 0) (at 101.9688 58.3406 0)
+      (effects (font (size 1.27 1.27)) (justify right) hide)
+    )
+  )
   (global_label "PLED1" (shape input) (at 44.45 69.85 270) (fields_autoplaced)
     (effects (font (size 1.27 1.27)) (justify right))
     (property "Intersheet References" "${INTERSHEET_REFS}" (id 0) (at 44.3706 78.1898 90)
+      (effects (font (size 1.27 1.27)) (justify right) hide)
+    )
+  )
+  (global_label "SCL" (shape input) (at 107.95 55.88 180) (fields_autoplaced)
+    (effects (font (size 1.27 1.27)) (justify right))
+    (property "Intersheet References" "${INTERSHEET_REFS}" (id 0) (at 102.0293 55.8006 0)
       (effects (font (size 1.27 1.27)) (justify right) hide)
     )
@@
     (pin "3")
   )
+  (symbol (lib_id "power:GND") (at 107.95 63.5 0) (unit 1)
+    (in_bom yes) (on_board yes) (fields_autoplaced)
+    (property "Reference" "#PWR070" (id 0) (at 107.95 69.85 0)
+      (effects (font (size 1.27 1.27)) hide)
+    )
+    (property "Value" "GND" (id 1) (at 107.95 68.58 0))
+    (property "Footprint" "" (id 2) (at 107.95 63.5 0)
+      (effects (font (size 1.27 1.27)) hide)
+    )
+    (property "Datasheet" "" (id 3) (at 107.95 63.5 0)
+      (effects (font (size 1.27 1.27)) hide)
+    )
+    (pin "1")
+  )
   (symbol (lib_id "power:GND") (at 33.02 62.23 0) (unit 1)
     (in_bom yes) (on_board yes) (fields_autoplaced)
@@
   (symbol (lib_id "power:GND") (at 107.95 31.75 0) (unit 1)
     (in_bom yes) (on_board yes) (fields_autoplaced)
-    (property "Reference" "#PWR068" (id 0) (at 107.95 38.1 0)
+    (property "Reference" "#PWR069" (id 0) (at 107.95 38.1 0)
       (effects (font (size 1.27 1.27)) hide)
     )
@@
   (symbol (lib_id "power:VBUS") (at 107.95 26.67 0) (unit 1)
     (in_bom yes) (on_board yes) (fields_autoplaced)
-    (property "Reference" "#PWR067" (id 0) (at 107.95 30.48 0)
+    (property "Reference" "#PWR068" (id 0) (at 107.95 30.48 0)
       (effects (font (size 1.27 1.27)) hide)
     )
@@
     (pin "2")
   )
+  (symbol (lib_id "Connector_Generic:Conn_01x04") (at 113.03 58.42 0) (unit 1)
+    (in_bom yes) (on_board yes) (fields_autoplaced)
+    (property "Reference" "J5" (id 0) (at 115.57 58.4199 0)
+      (effects (font (size 1.27 1.27)) (justify left))
+    )
+    (property "Value" "qwiic" (id 1) (at 115.57 60.9599 0)
+      (effects (font (size 1.27 1.27)) (justify left))
+    )
+    (property "Footprint" "Connector_JST:JST_SH_BM04B-SRSS-TB_1x04-1MP_P1.00mm_Vertical" (id 2) (at 113.03 58.42 0)
+      (effects (font (size 1.27 1.27)) hide)
+    )
+    (property "Datasheet" "~" (id 3) (at 113.03 58.42 0)
+      (effects (font (size 1.27 1.27)) hide)
+    )
+    (pin "1")
+    (pin "2")
+    (pin "3")
+    (pin "4")
+  )
   (symbol (lib_id "Device:R") (at 44.45 132.08 0) (unit 1)
     (in_bom yes) (on_board yes) (fields_autoplaced)
@@
       (effects (font (size 1.27 1.27)) hide)
     )
+    (pin "1")
+  )
+  (symbol (lib_id "power:+3.3V") (at 97.79 60.96 0) (unit 1)
+    (in_bom yes) (on_board yes) (fields_autoplaced)
+    (property "Reference" "#PWR067" (id 0) (at 97.79 64.77 0)
+      (effects (font (size 1.27 1.27)) hide)
+    )
+    (property "Value" "+3.3V" (id 1) (at 97.79 55.88 0))
+    (property "Footprint" "" (id 2) (at 97.79 60.96 0)
+      (effects (font (size 1.27 1.27)) hide)
+    )
+    (property "Datasheet" "" (id 3) (at 97.79 60.96 0)
+      (effects (font (size 1.27 1.27)) hide)
+    )

Commit message: Progress
Parts:
- J5: footprint Connector_JST:JST_SH_BM04B-SRSS-TB_1x04-1MP_P1.00mm_Vertical -> Connector_JST:JST_SH_SM04B-SRSS-TB_1x04-1MP_P1.00mm_Horizontal
Changed lines of the file:
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@@
       (effects (font (size 1.27 1.27)) (justify left))
     )
-    (property "Footprint" "Connector_JST:JST_SH_BM04B-SRSS-TB_1x04-1MP_P1.00mm_Vertical" (id 2) (at 113.03 58.42 0)
+    (property "Footprint" "Connector_JST:JST_SH_SM04B-SRSS-TB_1x04-1MP_P1.00mm_Horizontal" (id 2) (at 113.03 58.42 0)
       (effects (font (size 1.27 1.27)) hide)
     )

Commit message: a lot of Silkscreen work
Parts:
- D1, D2, D3, D4: footprint LED_SMD:LED_0805_2012Metric_Pad1.15x1.40mm_HandSolder -> OpenStick:LED_0805_2012Metric_Pad1.15x1.40mm_HandSolder
- R10, R7, R8, R9: footprint Resistor_SMD:R_0805_2012Metric_Pad1.20x1.40mm_HandSolder -> OpenStick:R_0805_2012Metric_Pad1.20x1.40mm_HandSolder
- renumbered J3 to J7, J4 to J8, J5 to J9
Changed lines of the file:
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@@
   (symbol (lib_id "power:GND") (at 22.86 30.48 0) (unit 1)
     (in_bom yes) (on_board yes) (fields_autoplaced)
-    (property "Reference" "#PWR062" (id 0) (at 22.86 36.83 0)
+    (property "Reference" "#PWR054" (id 0) (at 22.86 36.83 0)
       (effects (font (size 1.27 1.27)) hide)
     )
@@
   (symbol (lib_id "Connector_Generic:Conn_01x03") (at 38.1 30.48 0) (unit 1)
     (in_bom yes) (on_board yes) (fields_autoplaced)
-    (property "Reference" "J3" (id 0) (at 40.64 29.2099 0)
+    (property "Reference" "J7" (id 0) (at 40.64 29.2099 0)
       (effects (font (size 1.27 1.27)) (justify left))
     )
@@
   (symbol (lib_id "power:GND") (at 33.02 106.68 0) (unit 1)
     (in_bom yes) (on_board yes) (fields_autoplaced)
-    (property "Reference" "#PWR065" (id 0) (at 33.02 113.03 0)
+    (property "Reference" "#PWR057" (id 0) (at 33.02 113.03 0)
       (effects (font (size 1.27 1.27)) hide)
     )
@@
       (effects (font (size 1.27 1.27)) (justify left))
     )
-    (property "Footprint" "Resistor_SMD:R_0805_2012Metric_Pad1.20x1.40mm_HandSolder" (id 2) (at 42.672 66.04 90)
+    (property "Footprint" "OpenStick:R_0805_2012Metric_Pad1.20x1.40mm_HandSolder" (id 2) (at 42.672 66.04 90)
       (effects (font (size 1.27 1.27)) hide)
     )
@@
       (effects (font (size 1.27 1.27)) (justify left))
     )
-    (property "Footprint" "Resistor_SMD:R_0805_2012Metric_Pad1.20x1.40mm_HandSolder" (id 2) (at 42.672 90.17 90)
+    (property "Footprint" "OpenStick:R_0805_2012Metric_Pad1.20x1.40mm_HandSolder" (id 2) (at 42.672 90.17 90)
       (effects (font (size 1.27 1.27)) hide)
     )
@@
   (symbol (lib_id "Connector_Generic:Conn_01x03") (at 113.03 29.21 0) (unit 1)
     (in_bom yes) (on_board yes) (fields_autoplaced)
-    (property "Reference" "J4" (id 0) (at 115.57 27.9399 0)
+    (property "Reference" "J8" (id 0) (at 115.57 27.9399 0)
       (effects (font (size 1.27 1.27)) (justify left))
     )
@@
   (symbol (lib_id "power:GND") (at 107.95 63.5 0) (unit 1)
     (in_bom yes) (on_board yes) (fields_autoplaced)
-    (property "Reference" "#PWR070" (id 0) (at 107.95 69.85 0)
+    (property "Reference" "#PWR062" (id 0) (at 107.95 69.85 0)
       (effects (font (size 1.27 1.27)) hide)
     )
@@
   (symbol (lib_id "power:GND") (at 33.02 62.23 0) (unit 1)
     (in_bom yes) (on_board yes) (fields_autoplaced)
-    (property "Reference" "#PWR063" (id 0) (at 33.02 68.58 0)
+    (property "Reference" "#PWR055" (id 0) (at 33.02 68.58 0)
       (effects (font (size 1.27 1.27)) hide)
     )
@@
   (symbol (lib_id "power:GND") (at 107.95 31.75 0) (unit 1)
     (in_bom yes) (on_board yes) (fields_autoplaced)
-    (property "Reference" "#PWR069" (id 0) (at 107.95 38.1 0)
+    (property "Reference" "#PWR061" (id 0) (at 107.95 38.1 0)
       (effects (font (size 1.27 1.27)) hide)
     )
@@
   (symbol (lib_id "power:VBUS") (at 107.95 26.67 0) (unit 1)
     (in_bom yes) (on_board yes) (fields_autoplaced)
-    (property "Reference" "#PWR068" (id 0) (at 107.95 30.48 0)
+    (property "Reference" "#PWR060" (id 0) (at 107.95 30.48 0)
       (effects (font (size 1.27 1.27)) hide)
     )
@@
   (symbol (lib_id "power:GND") (at 33.02 86.36 0) (unit 1)
     (in_bom yes) (on_board yes) (fields_autoplaced)
-    (property "Reference" "#PWR064" (id 0) (at 33.02 92.71 0)
+    (property "Reference" "#PWR056" (id 0) (at 33.02 92.71 0)
       (effects (font (size 1.27 1.27)) hide)
     )
@@
     (property "Reference" "D3" (id 0) (at 39.0525 100.33 0))
     (property "Value" "PLED3" (id 1) (at 39.0525 102.87 0))
-    (property "Footprint" "LED_SMD:LED_0805_2012Metric_Pad1.15x1.40mm_HandSolder" (id 2) (at 40.64 106.68 0)
+    (property "Footprint" "OpenStick:LED_0805_2012Metric_Pad1.15x1.40mm_HandSolder" (id 2) (at 40.64 106.68 0)
       (effects (font (size 1.27 1.27)) hide)
     )
@@
     (property "Reference" "D1" (id 0) (at 39.0525 55.88 0))
     (property "Value" "PLED1" (id 1) (at 39.0525 58.42 0))
-    (property "Footprint" "LED_SMD:LED_0805_2012Metric_Pad1.15x1.40mm_HandSolder" (id 2) (at 40.64 62.23 0)
+    (property "Footprint" "OpenStick:LED_0805_2012Metric_Pad1.15x1.40mm_HandSolder" (id 2) (at 40.64 62.23 0)
       (effects (font (size 1.27 1.27)) hide)
     )
@@
   (symbol (lib_id "Connector_Generic:Conn_01x04") (at 113.03 58.42 0) (unit 1)
     (in_bom yes) (on_board yes) (fields_autoplaced)
-    (property "Reference" "J5" (id 0) (at 115.57 58.4199 0)
+    (property "Reference" "J9" (id 0) (at 115.57 58.4199 0)
       (effects (font (size 1.27 1.27)) (justify left))
     )
@@
       (effects (font (size 1.27 1.27)) (justify left))
     )
-    (property "Footprint" "Resistor_SMD:R_0805_2012Metric_Pad1.20x1.40mm_HandSolder" (id 2) (at 42.672 132.08 90)
+    (property "Footprint" "OpenStick:R_0805_2012Metric_Pad1.20x1.40mm_HandSolder" (id 2) (at 42.672 132.08 90)
       (effects (font (size 1.27 1.27)) hide)
     )
@@
       (effects (font (size 1.27 1.27)) (justify left))
     )
-    (property "Footprint" "Resistor_SMD:R_0805_2012Metric_Pad1.20x1.40mm_HandSolder" (id 2) (at 42.672 110.49 90)
+    (property "Footprint" "OpenStick:R_0805_2012Metric_Pad1.20x1.40mm_HandSolder" (id 2) (at 42.672 110.49 90)
       (effects (font (size 1.27 1.27)) hide)
     )
@@
   (symbol (lib_id "power:GND") (at 33.02 128.27 0) (unit 1)
     (in_bom yes) (on_board yes) (fields_autoplaced)
-    (property "Reference" "#PWR066" (id 0) (at 33.02 134.62 0)
+    (property "Reference" "#PWR058" (id 0) (at 33.02 134.62 0)
       (effects (font (size 1.27 1.27)) hide)
     )
@@
   (symbol (lib_id "power:+3.3V") (at 97.79 60.96 0) (unit 1)
     (in_bom yes) (on_board yes) (fields_autoplaced)
-    (property "Reference" "#PWR067" (id 0) (at 97.79 64.77 0)
+    (property "Reference" "#PWR059" (id 0) (at 97.79 64.77 0)
       (effects (font (size 1.27 1.27)) hide)
     )
@@
     (property "Reference" "D4" (id 0) (at 39.0525 121.92 0))
     (property "Value" "PLED4" (id 1) (at 39.0525 124.46 0))
-    (property "Footprint" "LED_SMD:LED_0805_2012Metric_Pad1.15x1.40mm_HandSolder" (id 2) (at 40.64 128.27 0)
+    (property "Footprint" "OpenStick:LED_0805_2012Metric_Pad1.15x1.40mm_HandSolder" (id 2) (at 40.64 128.27 0)
       (effects (font (size 1.27 1.27)) hide)
     )
@@
     (property "Reference" "D2" (id 0) (at 39.0525 80.01 0))
     (property "Value" "PLED2" (id 1) (at 39.0525 82.55 0))
-    (property "Footprint" "LED_SMD:LED_0805_2012Metric_Pad1.15x1.40mm_HandSolder" (id 2) (at 40.64 86.36 0)
-      (effects (font (size 1.27 1.27)) hide)
-    )
+    (property "Footprint" "OpenStick:LED_0805_2012Metric_Pad1.15x1.40mm_HandSolder" (id 2) (at 40.64 86.36 0)
+      (effects (font (size 1.27 1.27)) hide)
+    )
