File: GP2040-CE-DevBoard/pico.kicad_sch (KiCad schematic)
At the start: 3 parts

Commit message: Schematic nearly complete, PCB started
Parts:
- gave numbers to parts that had none: 3
Connections:
- net VSYS: no longer names the net of U1.39 (VSYS)
- no-connect marks 4 -> 5
Changed lines of the file:
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@@
   )
   (no_connect (at 213.36 92.71))
+  (no_connect (at 213.36 82.55))
   (no_connect (at 213.36 87.63))
   (no_connect (at 213.36 62.23))
@@
     )
   )
-  (global_label "VSYS" (shape bidirectional) (at 213.36 82.55 0) (fields_autoplaced)
-    (effects (font (size 1.27 1.27)) (justify left))
-    (property "Intersheet References" "${INTERSHEET_REFS}" (id 0) (at 220.3693 82.4706 0)
-      (effects (font (size 1.27 1.27)) (justify left) hide)
-    )
-  )
   (global_label "Select" (shape bidirectional) (at 86.36 62.23 180) (fields_autoplaced)
     (effects (font (size 1.27 1.27)) (justify right))
@@
   (symbol (lib_id "ul_SC0915:Raspbery Pi Pico") (at 86.36 46.99 0) (unit 1)
     (in_bom yes) (on_board yes) (fields_autoplaced)
-    (property "Reference" "U?" (id 0) (at 149.86 31.75 0)
+    (property "Reference" "U1" (id 0) (at 149.86 31.75 0)
       (effects (font (size 1.524 1.524)))
     )
@@
   (symbol (lib_id "power:GND") (at 220.98 46.99 0) (unit 1)
     (in_bom yes) (on_board yes) (fields_autoplaced)
-    (property "Reference" "#PWR?" (id 0) (at 220.98 53.34 0)
+    (property "Reference" "#PWR013" (id 0) (at 220.98 53.34 0)
       (effects (font (size 1.27 1.27)) hide)
     )
@@
   (symbol (lib_id "Device:R") (at 236.22 106.68 0) (unit 1)
     (in_bom yes) (on_board yes) (fields_autoplaced)
-    (property "Reference" "R?" (id 0) (at 238.76 105.4099 0)
+    (property "Reference" "R4" (id 0) (at 238.76 105.4099 0)
       (effects (font (size 1.27 1.27)) (justify left))
     )
@@
   (symbol (lib_id "power:+3.3V") (at 220.98 90.17 0) (unit 1)
     (in_bom yes) (on_board yes) (fields_autoplaced)
-    (property "Reference" "#PWR?" (id 0) (at 220.98 93.98 0)
+    (property "Reference" "#PWR014" (id 0) (at 220.98 93.98 0)
       (effects (font (size 1.27 1.27)) hide)
     )
@@
   (symbol (lib_id "power:GND") (at 215.9 85.09 0) (unit 1)
     (in_bom yes) (on_board yes) (fields_autoplaced)
-    (property "Reference" "#PWR?" (id 0) (at 215.9 91.44 0)
+    (property "Reference" "#PWR012" (id 0) (at 215.9 91.44 0)
       (effects (font (size 1.27 1.27)) hide)
     )
@@
   (symbol (lib_id "power:GND") (at 73.66 102.87 0) (unit 1)
     (in_bom yes) (on_board yes) (fields_autoplaced)
-    (property "Reference" "#PWR?" (id 0) (at 73.66 109.22 0)
+    (property "Reference" "#PWR07" (id 0) (at 73.66 109.22 0)
       (effects (font (size 1.27 1.27)) hide)
     )
@@
   (symbol (lib_id "power:GND") (at 76.2 77.47 0) (unit 1)
     (in_bom yes) (on_board yes) (fields_autoplaced)
-    (property "Reference" "#PWR?" (id 0) (at 76.2 83.82 0)
+    (property "Reference" "#PWR010" (id 0) (at 76.2 83.82 0)
       (effects (font (size 1.27 1.27)) hide)
     )
@@
   (symbol (lib_id "power:GND") (at 226.06 74.93 0) (unit 1)
     (in_bom yes) (on_board yes) (fields_autoplaced)
-    (property "Reference" "#PWR?" (id 0) (at 226.06 81.28 0)
+    (property "Reference" "#PWR016" (id 0) (at 226.06 81.28 0)
       (effects (font (size 1.27 1.27)) hide)
     )
@@
   (symbol (lib_id "power:+3.3V") (at 246.38 110.49 0) (unit 1)
     (in_bom yes) (on_board yes) (fields_autoplaced)
-    (property "Reference" "#PWR?" (id 0) (at 246.38 114.3 0)
+    (property "Reference" "#PWR020" (id 0) (at 246.38 114.3 0)
       (effects (font (size 1.27 1.27)) hide)
     )
@@
   (symbol (lib_id "Device:R") (at 227.33 109.22 0) (unit 1)
     (in_bom yes) (on_board yes) (fields_autoplaced)
-    (property "Reference" "R?" (id 0) (at 229.87 107.9499 0)
+    (property "Reference" "R3" (id 0) (at 229.87 107.9499 0)
       (effects (font (size 1.27 1.27)) (justify left))
     )
@@
   (symbol (lib_id "power:GND") (at 74.93 52.07 0) (unit 1)
     (in_bom yes) (on_board yes) (fields_autoplaced)
-    (property "Reference" "#PWR?" (id 0) (at 74.93 58.42 0)
+    (property "Reference" "#PWR08" (id 0) (at 74.93 58.42 0)
       (effects (font (size 1.27 1.27)) hide)
     )
@@
   (symbol (lib_id "power:GND") (at 76.2 90.17 0) (unit 1)
     (in_bom yes) (on_board yes) (fields_autoplaced)
-    (property "Reference" "#PWR?" (id 0) (at 76.2 96.52 0)
+    (property "Reference" "#PWR011" (id 0) (at 76.2 96.52 0)
       (effects (font (size 1.27 1.27)) hide)
     )
@@
   (symbol (lib_id "power:GND") (at 74.93 64.77 0) (unit 1)
     (in_bom yes) (on_board yes) (fields_autoplaced)
-    (property "Reference" "#PWR?" (id 0) (at 74.93 71.12 0)
+    (property "Reference" "#PWR09" (id 0) (at 74.93 71.12 0)
       (effects (font (size 1.27 1.27)) hide)
     )
@@
   (symbol (lib_id "power:GND") (at 223.52 110.49 0) (unit 1)
     (in_bom yes) (on_board yes) (fields_autoplaced)
-    (property "Reference" "#PWR?" (id 0) (at 223.52 116.84 0)
+    (property "Reference" "#PWR015" (id 0) (at 223.52 116.84 0)
       (effects (font (size 1.27 1.27)) hide)
     )
@@
   (symbol (lib_id "power:GND") (at 252.73 97.79 0) (unit 1)
     (in_bom yes) (on_board yes) (fields_autoplaced)
-    (property "Reference" "#PWR?" (id 0) (at 252.73 104.14 0)
+    (property "Reference" "#PWR021" (id 0) (at 252.73 104.14 0)
       (effects (font (size 1.27 1.27)) hide)
     )
@@
   (symbol (lib_id "power:VBUS") (at 233.68 80.01 0) (unit 1)
     (in_bom yes) (on_board yes) (fields_autoplaced)
-    (property "Reference" "#PWR?" (id 0) (at 233.68 83.82 0)
+    (property "Reference" "#PWR018" (id 0) (at 233.68 83.82 0)
       (effects (font (size 1.27 1.27)) hide)
     )
@@
   (symbol (lib_id "power:GND") (at 238.76 69.85 0) (unit 1)
     (in_bom yes) (on_board yes) (fields_autoplaced)
-    (property "Reference" "#PWR?" (id 0) (at 238.76 76.2 0)
+    (property "Reference" "#PWR019" (id 0) (at 238.76 76.2 0)
       (effects (font (size 1.27 1.27)) hide)
     )
@@
   (symbol (lib_id "power:+3.3V") (at 232.41 118.11 0) (unit 1)
     (in_bom yes) (on_board yes) (fields_autoplaced)
-    (property "Reference" "#PWR?" (id 0) (at 232.41 121.92 0)
-      (effects (font (size 1.27 1.27)) hide)
-    )
+    (property "Reference" "#PWR017" (id 0) (at 232.41 121.92 0)
+      (effects (font (size 1.27 1.27)) hide)
+    )

Commit message: Updating schema and PCB design
Connections:
- net 4K is gone; now on net PLED3: U1.19 (I2C1_SDA/SPI1_SCK/GP14)
- net Home is gone; now on net Right: U1.6 (UART1_TX/I2C0_SDA/SPI0_RX/GP4)
- net RSB is gone; now on net RGB: U1.29 (GP22)
- net Select is gone; now on net Left: U1.7 (UART1_RX/I2C0_SCL/SPI0_CSn/GP5)
- net Down: now also U1.5 (I2C1_SCL/SPI0_TX/GP3); no longer U1.4 (I2C1_SDA/SPI0_SCK/GP2)
- net Left: no longer U1.1 (UART0_TX/I2C0_SDA/SPI0_RX/GP0)
- net PLED1: now also U1.1 (UART0_TX/I2C0_SDA/SPI0_RX/GP0); no longer U1.21 (UART0_TX/I2C0_SDA/SPI0_RX/GP16)
- net PLED2: now also U1.2 (UART0_RX/I2C0_SCL/GPI0_CSn/GP1); no longer U1.22 (UART0_RX/I2C0_SCL/SPI0_CSn/GP17)
- net PLED3: no longer U1.24 (I2C1_SDA/SPI0_SCK/GP18)
- net PLED4: now also U1.20 (I2C1_SCL/SPI1_TX/GP15); no longer U1.25 (I2C1_SCL/SPI0_TX/GP19)
- net RGB: no longer U1.20 (I2C1_SCL/SPI1_TX/GP15)
- net Right: no longer U1.5 (I2C1_SCL/SPI0_TX/GP3)
- net Up: now also U1.4 (I2C1_SDA/SPI0_SCK/GP2); no longer U1.2 (UART0_RX/I2C0_SCL/GPI0_CSn/GP1)
- net 1K renamed B4
- net 1P renamed B2
- net 2K renamed R1
- net 2P renamed R2
- net 3K renamed L1
- net 3P renamed L2
- net 4P renamed B3
- net LSB renamed A2
- net Start renamed B1
- net TP renamed A1
- new net L3: U1.24 (I2C1_SDA/SPI0_SCK/GP18)
- new net R3: U1.25 (I2C1_SCL/SPI0_TX/GP19)
- new net S1: U1.21 (UART0_TX/I2C0_SDA/SPI0_RX/GP16)
- new net S2: U1.22 (UART0_RX/I2C0_SCL/SPI0_CSn/GP17)

Commit message: Progress
Parts:
- U1: footprint ul_SC0915:SC0915 -> OpenStick:Raspberry Pi Pico - pogo pin and screw mount
Connections:
- net B1: now also U1.11 (UART1_TX/I2C0_SDA/SPI1_RX/GP8); no longer U1.9 (I2C1_SDA/SPI0_SCK/GP6)
- net B2: now also U1.12 (UART1_RX/I2C0_SCL/SPI1_CSn/GP9); no longer U1.10 (I2C1_SCL/SPI0_TX/GP7)
- net B3: now also U1.16 (UART0_TX/I2C0_SDA/GPI1_RX/GP12); no longer U1.14 (I2C1_SDA/SPI1_SCK/GP10)
- net B4: now also U1.17 (UART0_RX/I2C0_SCL/SPI1_CSn/GP13); no longer U1.15 (I2C1_SCL/SPI1_TX/GP11)
- net Down: now also U1.7 (UART1_RX/I2C0_SCL/SPI0_CSn/GP5); no longer U1.5 (I2C1_SCL/SPI0_TX/GP3)
- net L1: now also U1.20 (I2C1_SCL/SPI1_TX/GP15); no longer U1.17 (UART0_RX/I2C0_SCL/SPI1_CSn/GP13)
- net L2: now also U1.15 (I2C1_SCL/SPI1_TX/GP11); no longer U1.12 (UART1_RX/I2C0_SCL/SPI1_CSn/GP9)
- net Left: now also U1.10 (I2C1_SCL/SPI0_TX/GP7); no longer U1.7 (UART1_RX/I2C0_SCL/SPI0_CSn/GP5)
- net PLED3: now also U1.4 (I2C1_SDA/SPI0_SCK/GP2); no longer U1.19 (I2C1_SDA/SPI1_SCK/GP14)
- net PLED4: now also U1.5 (I2C1_SCL/SPI0_TX/GP3); no longer U1.20 (I2C1_SCL/SPI1_TX/GP15)
- net R1: now also U1.19 (I2C1_SDA/SPI1_SCK/GP14); no longer U1.16 (UART0_TX/I2C0_SDA/GPI1_RX/GP12)
- net R2: now also U1.14 (I2C1_SDA/SPI1_SCK/GP10); no longer U1.11 (UART1_TX/I2C0_SDA/SPI1_RX/GP8)
- net Right: now also U1.9 (I2C1_SDA/SPI0_SCK/GP6); no longer U1.6 (UART1_TX/I2C0_SDA/SPI0_RX/GP4)
- net Up: now also U1.6 (UART1_TX/I2C0_SDA/SPI0_RX/GP4); no longer U1.4 (I2C1_SDA/SPI0_SCK/GP2)

Commit message: a lot of Silkscreen work
Parts:
- R3, R4: footprint Capacitor_SMD:C_0805_2012Metric_Pad1.18x1.45mm_HandSolder -> OpenStick:C_0805_2012Metric_Pad1.18x1.45mm_HandSolder
- U1: footprint OpenStick:Raspberry Pi Pico - pogo pin and screw mount -> ul_SC0915:Pico
Changed lines of the file:
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@@
       (effects (font (size 1.524 1.524)))
     )
-    (property "Footprint" "OpenStick:Raspberry Pi Pico - pogo pin and screw mount" (id 2) (at 149.86 40.894 0)
+    (property "Footprint" "ul_SC0915:Pico" (id 2) (at 149.86 40.894 0)
       (effects (font (size 1.524 1.524)) hide)
     )
@@
       (effects (font (size 1.27 1.27)) (justify left))
     )
-    (property "Footprint" "Capacitor_SMD:C_0805_2012Metric_Pad1.18x1.45mm_HandSolder" (id 2) (at 234.442 106.68 90)
+    (property "Footprint" "OpenStick:C_0805_2012Metric_Pad1.18x1.45mm_HandSolder" (id 2) (at 234.442 106.68 90)
       (effects (font (size 1.27 1.27)) hide)
     )
@@
   (symbol (lib_id "power:GND") (at 74.93 102.87 0) (unit 1)
     (in_bom yes) (on_board yes) (fields_autoplaced)
-    (property "Reference" "#PWR07" (id 0) (at 74.93 109.22 0)
+    (property "Reference" "#PWR011" (id 0) (at 74.93 109.22 0)
       (effects (font (size 1.27 1.27)) hide)
     )
@@
   (symbol (lib_id "power:GND") (at 74.93 77.47 0) (unit 1)
     (in_bom yes) (on_board yes) (fields_autoplaced)
-    (property "Reference" "#PWR010" (id 0) (at 74.93 83.82 0)
+    (property "Reference" "#PWR09" (id 0) (at 74.93 83.82 0)
       (effects (font (size 1.27 1.27)) hide)
     )
@@
       (effects (font (size 1.27 1.27)) (justify left))
     )
-    (property "Footprint" "Capacitor_SMD:C_0805_2012Metric_Pad1.18x1.45mm_HandSolder" (id 2) (at 225.552 109.22 90)
+    (property "Footprint" "OpenStick:C_0805_2012Metric_Pad1.18x1.45mm_HandSolder" (id 2) (at 225.552 109.22 90)
       (effects (font (size 1.27 1.27)) hide)
     )
@@
   (symbol (lib_id "power:GND") (at 74.93 52.07 0) (unit 1)
     (in_bom yes) (on_board yes) (fields_autoplaced)
-    (property "Reference" "#PWR08" (id 0) (at 74.93 58.42 0)
+    (property "Reference" "#PWR07" (id 0) (at 74.93 58.42 0)
       (effects (font (size 1.27 1.27)) hide)
     )
@@
   (symbol (lib_id "power:GND") (at 74.93 90.17 0) (unit 1)
     (in_bom yes) (on_board yes) (fields_autoplaced)
-    (property "Reference" "#PWR011" (id 0) (at 74.93 96.52 0)
+    (property "Reference" "#PWR010" (id 0) (at 74.93 96.52 0)
       (effects (font (size 1.27 1.27)) hide)
     )
@@
   (symbol (lib_id "power:GND") (at 74.93 64.77 0) (unit 1)
     (in_bom yes) (on_board yes) (fields_autoplaced)
-    (property "Reference" "#PWR09" (id 0) (at 74.93 71.12 0)
-      (effects (font (size 1.27 1.27)) hide)
-    )
+    (property "Reference" "#PWR08" (id 0) (at 74.93 71.12 0)
+      (effects (font (size 1.27 1.27)) hide)
+    )
